Commit message: tfからcollsionを指定する際にURDFを読み込めるように変更

File: collision_objects/ic120_description/urdf/ic120.urdf (robot description, URDF)
Before this commit: robot ic120, 13 links, 12 joints
Links:
- link body_link: geometry collision mesh filename=package://ic120_description/meshes/ic120-body.dae; visual mesh filename=package://ic120_description/meshes/ic120-body.dae
- link cylinder_head_link: geometry collision mesh filename=package://ic120_description/meshes/ic120-cylinder1.dae; visual mesh filename=package://ic120_description/meshes/ic120-cylinder1.dae
- link cylinder_rod_link: geometry collision mesh filename=package://ic120_description/meshes/ic120-cylinder2.dae; visual mesh filename=package://ic120_description/meshes/ic120-cylinder2.dae
- link vessel_pin_link: geometry collision mesh filename=package://ic120_description/meshes/ic120-vessel.dae; visual mesh filename=package://ic120_description/meshes/ic120-vessel.dae
