Commit message: experiment20250821

File: collision_objects/mst2200vd_description/urdf/mst2200vd.urdf (robot description, URDF)
Before this commit: robot mst2200vd, 6 links, 5 joints
Links:
- link body_link: geometry collision mesh filename=package://mst2200vd_description/meshes/mst2200vd-body.dae; visual mesh filename=package://mst2200vd_description/meshes/mst2200vd-body.dae
- link track_link: geometry collision mesh filename=package://mst2200vd_description/meshes/mst2200vd-crawler.dae; visual mesh filename=package://mst2200vd_description/meshes/mst2200vd-crawler.dae
- link vessel_cylinder_link: geometry collision mesh filename=package://mst2200vd_description/meshes/mst2200vd-vessel_cyl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; visual mesh filename=package://mst2200vd_description/meshes/mst2200vd-vessel_cyl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
- link vessel_link: geometry collision mesh filename=package://mst2200vd_description/meshes/mst2200vd-vessel.dae; visual mesh filename=package://mst2200vd_description/meshes/mst2200vd-vessel.dae
- link vessel_rod_link: geometry collision mesh filename=package://mst2200vd_description/meshes/mst2200vd-vessel_rod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; visual mesh filename=package://mst2200vd_description/meshes/mst2200vd-vessel_rod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
