Commit message: demo202508

File: collision_objects/mst110cr_description/urdf/mst110cr.urdf (robot description, URDF)
Before this commit: robot mst2200vd, 6 links, 5 joints
Links:
- link body_link: geometry collision mesh filename=package://mst110cr_description/meshes/mst110cr-body.dae; visual mesh filename=package://mst110cr_description/meshes/mst110cr-body.dae
- link track_link: geometry collision mesh filename=package://mst110cr_description/meshes/mst110cr-crawler.dae; visual mesh filename=package://mst110cr_description/meshes/mst110cr-crawler.dae
- link vessel_cylinder_link: geometry collision mesh filename=package://mst110cr_description/meshes/mst110cr-vessel_cylin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; visual mesh filename=package://mst110cr_description/meshes/mst110cr-vessel_cylin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
- link vessel_link: geometry collision mesh filename=package://mst110cr_description/meshes/mst110cr-vessel.dae; visual mesh filename=package://mst110cr_description/meshes/mst110cr-vessel.dae
- link vessel_rod_link: geometry collision mesh filename=package://mst110cr_description/meshes/mst110cr-vessel_rod.d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; visual mesh filename=package://mst110cr_description/meshes/mst110cr-vessel_rod.d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
